File: gamepad.sch (KiCad schematic (older format))
At the start: 19 parts, among them SW1 Elastomer SW, SW10 Elastomer SW, SW11 B3F-3000, SW12 B3F-3000, SW2 Elastomer SW, SW3 Elastomer SW, SW4 Elastomer SW, SW5 Elastomer SW, SW6 Elastomer SW, SW7 Elastomer SW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

Commit message: finished layout
Parts:
- SW1, SW10, SW2, SW3, SW4, SW5, SW6, SW7, SW8, SW9: footprint (none) -> gamepad:8mm_elastomer_button
- SW11, SW12: footprint (none) -> gamepad:B3F-3000
Changed lines of the file:
@@
 F 0 "SW1" H 7350 3035 50  0000 C CNN
 F 1 "Elastomer SW" H 7350 2944 50  0000 C CNN
-F 2 "" H 7350 2950 50  0001 C CNN
+F 2 "gamepad:8mm_elastomer_button" H 7350 2950 50  0001 C CNN
 F 3 "" H 7350 2950 50  0001 C CNN
 	1    7350 2750
@@
 F 0 "SW2" H 8250 3035 50  0000 C CNN
 F 1 "Elastomer SW" H 8250 2944 50  0000 C CNN
-F 2 "" H 8250 2950 50  0001 C CNN
+F 2 "gamepad:8mm_elastomer_button" H 8250 2950 50  0001 C CNN
 F 3 "" H 8250 2950 50  0001 C CNN
 	1    8250 2750
@@
 F 0 "SW3" H 7350 3435 50  0000 C CNN
 F 1 "Elastomer SW" H 7350 3344 50  0000 C CNN
-F 2 "" H 7350 3350 50  0001 C CNN
+F 2 "gamepad:8mm_elastomer_button" H 7350 3350 50  0001 C CNN
 F 3 "" H 7350 3350 50  0001 C CNN
 	1    7350 3150
@@
 F 0 "SW4" H 8250 3435 50  0000 C CNN
 F 1 "Elastomer SW" H 8250 3344 50  0000 C CNN
-F 2 "" H 8250 3350 50  0001 C CNN
+F 2 "gamepad:8mm_elastomer_button" H 8250 3350 50  0001 C CNN
 F 3 "" H 8250 3350 50  0001 C CNN
 	1    8250 3150
@@
 F 0 "SW5" H 7350 3835 50  0000 C CNN
 F 1 "Elastomer SW" H 7350 3744 50  0000 C CNN
-F 2 "" H 7350 3750 50  0001 C CNN
+F 2 "gamepad:8mm_elastomer_button" H 7350 3750 50  0001 C CNN
 F 3 "" H 7350 3750 50  0001 C CNN
 	1    7350 3550
@@
 F 0 "SW6" H 8250 3835 50  0000 C CNN
 F 1 "Elastomer SW" H 8250 3744 50  0000 C CNN
-F 2 "" H 8250 3750 50  0001 C CNN
+F 2 "gamepad:8mm_elastomer_button" H 8250 3750 50  0001 C CNN
 F 3 "" H 8250 3750 50  0001 C CNN
 	1    8250 3550
@@
 F 0 "SW7" H 7350 4235 50  0000 C CNN
 F 1 "Elastomer SW" H 7350 4144 50  0000 C CNN
-F 2 "" H 7350 4150 50  0001 C CNN
+F 2 "gamepad:8mm_elastomer_button" H 7350 4150 50  0001 C CNN
 F 3 "" H 7350 4150 50  0001 C CNN
 	1    7350 3950
@@
 F 0 "SW8" H 8250 4235 50  0000 C CNN
 F 1 "Elastomer SW" H 8250 4144 50  0000 C CNN
-F 2 "" H 8250 4150 50  0001 C CNN
+F 2 "gamepad:8mm_elastomer_button" H 8250 4150 50  0001 C CNN
 F 3 "" H 8250 4150 50  0001 C CNN
 	1    8250 3950
@@
 F 0 "SW9" H 7350 4635 50  0000 C CNN
 F 1 "Elastomer SW" H 7350 4544 50  0000 C CNN
-F 2 "" H 7350 4550 50  0001 C CNN
+F 2 "gamepad:8mm_elastomer_button" H 7350 4550 50  0001 C CNN
 F 3 "" H 7350 4550 50  0001 C CNN
 	1    7350 4350
@@
 F 0 "SW10" H 8250 4635 50  0000 C CNN
 F 1 "Elastomer SW" H 8250 4544 50  0000 C CNN
-F 2 "" H 8250 4550 50  0001 C CNN
+F 2 "gamepad:8mm_elastomer_button" H 8250 4550 50  0001 C CNN
 F 3 "" H 8250 4550 50  0001 C CNN
 	1    8250 4350
@@
 F 0 "SW11" H 7350 5035 50  0000 C CNN
 F 1 "B3F-3000" H 7350 4944 50  0000 C CNN
-F 2 "" H 7350 4950 50  0001 C CNN
+F 2 "gamepad:B3F-3000" H 7350 4950 50  0001 C CNN
 F 3 "" H 7350 4950 50  0001 C CNN
 	1    7350 4750
@@
 F 0 "SW12" H 8250 5035 50  0000 C CNN
 F 1 "B3F-3000" H 8250 4944 50  0000 C CNN
-F 2 "" H 8250 4950 50  0001 C CNN
+F 2 "gamepad:B3F-3000" H 8250 4950 50  0001 C CNN
 F 3 "" H 8250 4950 50  0001 C CNN
 	1    8250 4750
