File: gamepad.kicad_pcb (KiCad board)
At the start: 2 copper layers, 139 x 61 mm, 19 parts, among them SW1 Elastomer Switch, SW10 Elastomer Switch, SW11 Elastomer Switch, SW12 Elastomer Switch, SW2 Elastomer Switch, SW3 Elastomer Switch, SW4 Elastomer Switch, SW5 B3F-3000, SW6 B3F-3000, SW7 Elastomer Switch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

Commit message: finished layout
Routing:
- net /rbump: track 0.00 -> 105.1 mm, vias 0 -> 2
- net /left: track 0.00 -> 100.7 mm, vias 0 -> 1
- net /3V3: track 0.00 -> 93.8 mm
- net /x: track 0.00 -> 91.4 mm, vias 0 -> 1
- net /lbump: track 0.00 -> 83.6 mm
- net /up: track 0.00 -> 70.7 mm, vias 0 -> 1
- net /5V: track 0.00 -> 55.6 mm
- net /right: track 0.00 -> 53.4 mm, vias 0 -> 1
- net /SCK: track 0.00 -> 51.5 mm
- net /RT_CS: track 0.00 -> 50.5 mm
- net /EECLK: track 0.00 -> 50.5 mm
- net /MOSI: track 0.00 -> 50.5 mm
- net /SDA: track 0.00 -> 50.4 mm
- net /GPIO22: track 0.00 -> 50.4 mm
- net /EEDATA: track 0.00 -> 50.4 mm
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
Commit message: fixed oopsy whoopsy
Routing:
- net GND: track 0.00 -> 6.13 mm
Changed lines of the file:
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@@
     (thickness 1.6)
     (drawings 12)
-    (tracks 191)
+    (tracks 195)
     (zones 0)
     (modules 19)
@@
   (gr_line (start 93 72.5) (end 93 122.5) (layer Dwgs.User) (width 0.2))
   (gr_line (start 96 69.5) (end 175.5 69.5) (layer Dwgs.User) (width 0.2))
+  (segment (start 164.170001 122.390001) (end 165.02 123.24) (width 0.254) (layer Top) (net 1))
+  (segment (start 163.68 121.9) (end 164.170001 122.390001) (width 0.254) (layer Top) (net 1))
+  (segment (start 159.94 120.7) (end 161.14 121.9) (width 0.254) (layer Top) (net 1))
+  (segment (start 161.14 121.9) (end 163.68 121.9) (width 0.254) (layer Top) (net 1))
   (via (at 126.9 94.3) (size 1.27) (drill 1.016) (layers Top Bottom) (net 2))
   (segment (start 126.92 120.7) (end 126.92 94.32) (width 0.254) (layer Bottom) (net 2))
