File: gamepad.kicad_pcb (KiCad board)
At the start: 2 copper layers, 139 x 61 mm, 19 parts, among them SW1 Elastomer Switch, SW10 Elastomer Switch, SW11 Elastomer Switch, SW12 Elastomer Switch, SW2 Elastomer Switch, SW3 Elastomer Switch, SW4 Elastomer Switch, SW5 B3F-3000, SW6 B3F-3000, SW7 Elastomer Switch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

Commit message: Finalized Rev B
Parts:
- SW1, SW10, SW2, SW3, SW4, SW7, SW8, SW9: value Elastomer Switch -> Elastomer SW; footprint Button_Switch_THT:SW_PUSH_6mm_H8mm -> gamepad:8mm_elastomer_button
- SW11, SW12: value Elastomer Switch -> B3F-3000; footprint Button_Switch_THT:SW_PUSH_6mm_H8mm -> gamepad:B3F-3000; moved to B.Cu
- SW5, SW6: value B3F-3000 -> Elastomer SW; footprint gamepad:B3F-3000 -> gamepad:8mm_elastomer_button; moved to F.Cu
- moved SW6 41.3 mm to (145.6, 95.5)
- moved SW5 41.3 mm to (126.2, 95.5)
- moved SW12 39.7 mm to (175.0, 66.0)
- moved SW11 33.0 mm to (96.8, 66.0)
- moved SW3 13.3 mm to (96.8, 103.0)
- moved SW4 9.03 mm to (86.8, 95.5)
- moved SW2 6.91 mm to (106.8, 95.5)
- moved SW9 6.73 mm to (185.0, 95.5)
- moved SW7 4.65 mm to (175.0, 88.0)
- moved SW1 3.67 mm to (96.8, 88.0)
- moved SW8 3.54 mm to (175.0, 103.0)
- moved SW10 2.02 mm to (165.0, 95.5)
- moved JP1 0.40 mm to (146.0, 73.0)
Connections:
- SW10 pad 1: /y -> GND
- SW10 pad 2: GND -> /select
- SW11 pad 1: /start -> /lbump
- SW12 pad 1: /select -> GND
- SW12 pad 2: GND -> /rbump
- SW2 pad 1: /right -> GND
- SW2 pad 2: GND -> /right
- SW4 pad 1: /down -> GND
- SW4 pad 2: GND -> /down
- SW5 pad 1: /lbump -> /x
- SW6 pad 2: /rbump -> /b
- SW7 pad 1: /x -> /a
- SW8 pad 1: /b -> GND
- SW8 pad 2: GND -> /y
- SW9 pad 1: /a -> /start
Routing:
- net GND: track 6.13 -> 139.6 mm
- net /x: track 91.4 -> 47.3 mm
- net /start: track 42.2 -> 85.9 mm, vias 0 -> 1
- net /b: track 39.3 -> 69.1 mm
- net /down: track 48.7 -> 64.2 mm
- net /left: track 100.7 -> 89.0 mm
- net /lbump: track 83.6 -> 94.7 mm, vias 0 -> 1
- net /right: track 53.4 -> 42.7 mm
- net /select: track 47.6 -> 56.6 mm
- net /SDA: track 50.4 -> 54.0 mm
- net /3V3: track 93.8 -> 97.4 mm, vias 0 -> 1
- net /rbump: track 105.1 -> 101.8 mm, vias 2 -> 1
- net /a: track 49.0 -> 51.7 mm
- net /5V: track 55.6 -> 57.2 mm, vias 0 -> 1
- net /SCK: track 51.5 -> 50.0 mm
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- added copper zone on B.Cu, net GND
- removed copper zone on F.Cu, net GND
Other:
- board text added: "Rev B"
- board text added: "Spark Gamepad"
